File: hardware/pcb/Student Remote.kicad_sch (KiCad schematic)
At the start: 57 parts, among them J1 Conn_01x13_Pin, J2 Conn_01x13_Pin, J3 Conn_01x02_Pin, J4 Conn_01x02_Pin, Q1 AO3400A, Q2 AO3401A, SW1 SW_Push, SW10 SW_Push, SW11 SW_Push, SW12 SW_Push, SW13 SW_Wuerth_450301014042, SW2 SW_Push, SW3 SW_Push, SW4 SW_Push, SW5 SW_Push, SW6 SW_Push, SW7 SW_Push, SW8 SW_Push, SW9 SW_Push, U1 74HC595, U2 74HC595, U3 HDSP-7501, U4 HDSP-7501

Commit message: Schematic: 74HC595 pin 12 RCLK to lat, pin 10 SRCLR to 3V
Connections:
- net 3v: now also U1.10 (~{SRCLR}), U2.10 (~{SRCLR})
- net GND: no longer U1.12 (RCLK), U2.12 (RCLK)
- net lat: now also U1.12 (RCLK), U2.12 (RCLK); no longer U1.10 (~{SRCLR}), U2.10 (~{SRCLR})
Changed lines of the file:
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@@
 	)
 	(junction
-		(at 217.17 40.64)
-		(diameter 0)
-		(color 0 0 0 0)
-	)
-	(junction
 		(at 160.02 118.11)
 		(diameter 0)
@@
 	)
 	(junction
-		(at 217.17 87.63)
-		(diameter 0)
-		(color 0 0 0 0)
-	)
-	(junction
 		(at 115.57 44.45)
 		(diameter 0)
@@
 	)
 	(junction
-		(at 210.82 35.56)
-		(diameter 0)
-		(color 0 0 0 0)
-	)
-	(junction
 		(at 128.27 52.07)
 		(diameter 0)
@@
 	(wire
 		(pts
-			(xy 219.71 85.09) (xy 217.17 85.09)
-		)
-		(stroke
-			(width 0)
-			(type default)
-		)
-	)
-	(wire
-		(pts
 			(xy 240.03 80.01) (xy 254 80.01)
 		)
@@
 	(wire
 		(pts
-			(xy 209.55 35.56) (xy 210.82 35.56)
-		)
-		(stroke
-			(width 0)
-			(type default)
-		)
-	)
-	(wire
-		(pts
-			(xy 210.82 33.02) (xy 210.82 35.56)
-		)
-		(stroke
-			(width 0)
-			(type default)
-		)
-	)
-	(wire
-		(pts
 			(xy 90.17 149.86) (xy 93.98 149.86)
 		)
@@
 	(wire
 		(pts
-			(xy 219.71 33.02) (xy 210.82 33.02)
-		)
-		(stroke
-			(width 0)
-			(type default)
-		)
-	)
-	(wire
-		(pts
 			(xy 160.02 125.73) (xy 160.02 128.27)
 		)
@@
 	(wire
 		(pts
-			(xy 210.82 80.01) (xy 219.71 80.01)
-		)
-		(stroke
-			(width 0)
-			(type default)
-		)
-	)
-	(wire
-		(pts
-			(xy 210.82 35.56) (xy 210.82 80.01)
-		)
-		(stroke
-			(width 0)
-			(type default)
-		)
-	)
-	(wire
-		(pts
 			(xy 115.57 59.69) (xy 132.08 59.69)
 		)
@@
 	(wire
 		(pts
-			(xy 217.17 38.1) (xy 217.17 40.64)
-		)
-		(stroke
-			(width 0)
-			(type default)
-		)
-	)
-	(wire
-		(pts
 			(xy 144.78 36.83) (xy 144.78 52.07)
 		)
@@
 	(wire
 		(pts
-			(xy 217.17 85.09) (xy 217.17 87.63)
-		)
-		(stroke
-			(width 0)
-			(type default)
-		)
-	)
-	(wire
-		(pts
 			(xy 161.29 36.83) (xy 161.29 52.07)
 		)
@@
 	(wire
 		(pts
-			(xy 219.71 38.1) (xy 217.17 38.1)
-		)
-		(stroke
-			(width 0)
-			(type default)
-		)
-	)
-	(wire
-		(pts
 			(xy 115.57 44.45) (xy 132.08 44.45)
 		)
@@
 		)
 	)
-	(global_label "lat"
-		(shape input)
-		(at 209.55 35.56 180)
-		(fields_autoplaced yes)
-		(effects
-			(font
-				(size 1.27 1.27)
-			)
-			(justify right)
-		)
-		(property "Intersheetrefs" "${INTERSHEET_REFS}"
-			(at 204.0249 35.56 0)
-			(effects
-				(font
-					(size 1.27 1.27)
-				)
-				(justify right)
-				(hide yes)
-			)
-		)
-	)
 	(global_label "mot"
 		(shape input)
@@
 			)
 		)
+	)
+	(wire
+		(pts
+			(xy 209.55 33.02) (xy 219.71 33.02)
+		)
+		(stroke
+			(width 0)
+			(type default)
+		)
+	)
+	(global_label "3v"
+		(shape input)
+		(at 209.55 33.02 180)
+		(fields_autoplaced yes)
+		(effects
+			(font
+				(size 1.27 1.27)
+			)
+			(justify right)
+		)
+		(property "Intersheetrefs" "${INTERSHEET_REFS}"
+			(at 204.3877 33.02 0)
+			(effects
+				(font
+					(size 1.27 1.27)
+				)
+				(justify right)
+				(hide yes)
+			)
+		)
+	)
+	(wire
+		(pts
+			(xy 209.55 38.1) (xy 219.71 38.1)
+		)
+		(stroke
+			(width 0)
+			(type default)
+		)
+	)
+	(global_label "lat"
+		(shape input)
+		(at 209.55 38.1 180)
+		(fields_autoplaced yes)
+		(effects
+			(font
+				(size 1.27 1.27)
+			)
+			(justify right)
+		)
+		(property "Intersheetrefs" "${INTERSHEET_REFS}"
+			(at 204.0249 38.1 0)
+			(effects
+				(font
+					(size 1.27 1.27)
+				)
+				(justify right)
+				(hide yes)
+			)
+		)
+	)
+	(wire
+		(pts
+			(xy 209.55 80.01) (xy 219.71 80.01)
+		)
+		(stroke
+			(width 0)
+			(type default)
+		)
+	)
+	(global_label "3v"
+		(shape input)
+		(at 209.55 80.01 180)
+		(fields_autoplaced yes)
+		(effects
+			(font
+				(size 1.27 1.27)
+			)
+			(justify right)
+		)
+		(property "Intersheetrefs" "${INTERSHEET_REFS}"
+			(at 204.3877 80.01 0)
+			(effects
+				(font
+					(size 1.27 1.27)
+				)
+				(justify right)
+				(hide yes)
+			)
+		)
+	)
+	(wire
+		(pts
+			(xy 209.55 85.09) (xy 219.71 85.09)
+		)
+		(stroke
+			(width 0)
+			(type default)
+		)
+	)
+	(global_label "lat"
+		(shape input)
+		(at 209.55 85.09 180)
+		(fields_autoplaced yes)
+		(effects
+			(font
+				(size 1.27 1.27)
+			)
+			(justify right)
+		)
+		(property "Intersheetrefs" "${INTERSHEET_REFS}"
+			(at 204.0249 85.09 0)
+			(effects
+				(font
+					(size 1.27 1.27)
+				)
+				(justify right)
+				(hide yes)
+			)
+		)
